File: hardware/Arduino_Nano_LCC_Boosters/can_interface.kicad_sch (KiCad schematic)
At the start: 3 parts, among them U11 MCP2515-xSO, U40 MCP2562-E-SN, Y1 16.0 MHz, 22pF

Commit message: Started placement and routing
Parts:
- Y1: footprint (none) -> Crystal:Crystal_HC49-U-3Pin_Vertical
Changed lines of the file:
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@@
 			)
 		)
-		(property "Footprint" ""
+		(property "Footprint" "Crystal:Crystal_HC49-U-3Pin_Vertical"
 			(at 106.68 98.425 0)
 			(effects
