File: hardware/Arduino_Nano_LCC_Boosters/Arduino_Nano_LCC_Boosters.kicad_pcb (KiCad board)
At the start: 2 copper layers, 213.4 x 137.2 mm, 134 parts, among them J1 Screw_Terminal_01x12, J2 RJ45_LED_Shielded_x2, J3 Barrel_Jack_MountingPin, J4 Screw_Terminal_01x12, Q1 AO3400A, Q2 AO3400A, Q3 AO3400A, Q4 AO3400A, Q5 AO3400A, Q6 AO3400A, Q7 AO3400A, Q8 AO3400A, SW1 SW_Push, SW2 SW_Push, SW3 SW_Slide_DPDT, U1 DRV8874PWPR, U10 DRV8874PWPR, U11 MCP2515-xSO, U12 7410, U13 7410, U14 7410, U15 DRV8874PWPR, U16 7404, U17 7410, U18 7410, U2 7410, U20 DRV8874PWPR, U21 MCP2515-xSO, U23 7404, U24 7410, U25 7410, U26 7410, U27 DRV8874PWPR, U28 7410, U29 7410, U3 7410, U30 7410, U31 DRV8874PWPR, U32 7410, U33 7410, U34 7410, U35 DRV8874PWPR, U36 7404, U37 7410, U38 7410, U39 DRV8874PWPR, U4 7410, U40 MCP2562-E-SN, U41 MCP2562-E-SN, U5 7404, U6 ACPL-214-500E, U7 7410, U8 7410, U9 7410, Y1 16.0 MHz, 22pF, Y2 16.0 MHz, 22pF

Commit message: Switch to single Arduino per board
Parts:
- removed the J1 at (22.9, 41.9)
- removed the R1 at (123.1, 38.0)
- removed the R2 at (64.2, 105.8)
- removed the R3 at (127.9, 38.0)
- removed the R4 at (132.7, 38.0)
- added C49: C22n, Capacitor_SMD:C_1206_3216Metric_Pad1.33x1.80mm_HandSolder, F.Cu at (-136.5, -97.5)
- added C50: C22n, Capacitor_SMD:C_1206_3216Metric_Pad1.33x1.80mm_HandSolder, F.Cu at (-136.5, -94.1)
- added C51: C100n, Capacitor_SMD:C_1206_3216Metric_Pad1.33x1.80mm_HandSolder, F.Cu at (-94.6, -124.3)
- added C52: C100n, Capacitor_SMD:C_1206_3216Metric_Pad1.33x1.80mm_HandSolder, F.Cu at (-94.6, -120.9)
- added C53: C100n, Capacitor_SMD:C_1206_3216Metric_Pad1.33x1.80mm_HandSolder, F.Cu at (-94.6, -117.6)
- added C54: C100n, Capacitor_SMD:C_1206_3216Metric_Pad1.33x1.80mm_HandSolder, F.Cu at (-94.6, -114.2)
- added C55: C100n, Capacitor_SMD:C_1206_3216Metric_Pad1.33x1.80mm_HandSolder, F.Cu at (-94.6, -110.9)
- added C56: C100n, Capacitor_SMD:C_1206_3216Metric_Pad1.33x1.80mm_HandSolder, F.Cu at (-94.6, -107.5)
- added C57: C10u, Capacitor_SMD:C_1206_3216Metric_Pad1.33x1.80mm_HandSolder, F.Cu at (-94.6, -104.2)
- added C58: C100n, Capacitor_SMD:C_1206_3216Metric_Pad1.33x1.80mm_HandSolder, F.Cu at (-94.6, -100.8)
- added C59: C22n, Capacitor_SMD:C_1206_3216Metric_Pad1.33x1.80mm_HandSolder, F.Cu at (-94.6, -97.5)
- added C60: C22n, Capacitor_SMD:C_1206_3216Metric_Pad1.33x1.80mm_HandSolder, F.Cu at (-94.6, -94.1)
- added C61: C100n, Capacitor_SMD:C_1206_3216Metric_Pad1.33x1.80mm_HandSolder, F.Cu at (-52.8, -159.8)
- added C62: C100n, Capacitor_SMD:C_1206_3216Metric_Pad1.33x1.80mm_HandSolder, F.Cu at (-52.8, -156.4)
- added C63: C100n, Capacitor_SMD:C_1206_3216Metric_Pad1.33x1.80mm_HandSolder, F.Cu at (-52.8, -153.1)
- added C64: C100n, Capacitor_SMD:C_1206_3216Metric_Pad1.33x1.80mm_HandSolder, F.Cu at (-52.8, -149.7)
- added C65: C100n, Capacitor_SMD:C_1206_3216Metric_Pad1.33x1.80mm_HandSolder, F.Cu at (-52.8, -146.4)
- added C66: C100n, Capacitor_SMD:C_1206_3216Metric_Pad1.33x1.80mm_HandSolder, F.Cu at (-52.8, -143.0)
- added C67: C10u, Capacitor_SMD:C_1206_3216Metric_Pad1.33x1.80mm_HandSolder, F.Cu at (-52.8, -139.7)
- added C68: C100n, Capacitor_SMD:C_1206_3216Metric_Pad1.33x1.80mm_HandSolder, F.Cu at (-52.8, -136.3)
- added C69: C22n, Capacitor_SMD:C_1206_3216Metric_Pad1.33x1.80mm_HandSolder, F.Cu at (-52.8, -133.0)
- added C70: C22n, Capacitor_SMD:C_1206_3216Metric_Pad1.33x1.80mm_HandSolder, F.Cu at (-52.8, -129.6)
- added C71: C100n, Capacitor_SMD:C_1206_3216Metric_Pad1.33x1.80mm_HandSolder, F.Cu at (-94.6, -88.8)
- added C72: C100n, Capacitor_SMD:C_1206_3216Metric_Pad1.33x1.80mm_HandSolder, F.Cu at (-94.6, -85.4)
- added C73: C100n, Capacitor_SMD:C_1206_3216Metric_Pad1.33x1.80mm_HandSolder, F.Cu at (-94.6, -82.1)
- added C74: C100n, Capacitor_SMD:C_1206_3216Metric_Pad1.33x1.80mm_HandSolder, F.Cu at (-94.6, -78.7)
- added C75: C100n, Capacitor_SMD:C_1206_3216Metric_Pad1.33x1.80mm_HandSolder, F.Cu at (-94.6, -75.4)
- added C76: C100n, Capacitor_SMD:C_1206_3216Metric_Pad1.33x1.80mm_HandSolder, F.Cu at (-94.6, -72.0)
- added C77: C10u, Capacitor_SMD:C_1206_3216Metric_Pad1.33x1.80mm_HandSolder, F.Cu at (-94.6, -68.7)
- added C78: C100n, Capacitor_SMD:C_1206_3216Metric_Pad1.33x1.80mm_HandSolder, F.Cu at (-94.6, -65.3)
- added C79: C22n, Capacitor_SMD:C_1206_3216Metric_Pad1.33x1.80mm_HandSolder, F.Cu at (-94.6, -62.0)
- added C80: C22n, Capacitor_SMD:C_1206_3216Metric_Pad1.33x1.80mm_HandSolder, F.Cu at (-94.6, -58.6)
- added J2: Screw_Terminal_01x08, TerminalBlock_Phoenix:TerminalBlock_Phoenix_MKDS-1,5-8_1x08_P5.00mm_Horizontal, F.Cu at (19.0, 46.1)
- added J3: Screw_Terminal_01x02, TerminalBlock_Phoenix:TerminalBlock_Phoenix_MKDS-1,5-2_1x02_P5.00mm_Horizontal, F.Cu at (19.1, 19.3)
- added J5: Screw_Terminal_01x08, TerminalBlock_Phoenix:TerminalBlock_Phoenix_MKDS-1,5-8_1x08_P5.00mm_Horizontal, F.Cu at (19.0, 99.7)
- added R13: R732, Resistor_SMD:R_0815_2038Metric_Pad1.20x4.05mm_HandSolder, F.Cu at (-113.1, -147.1)
- added R14: R47k, Resistor_SMD:R_0815_2038Metric_Pad1.20x4.05mm_HandSolder, F.Cu at (-80.9, -147.1)
- added R15: R1k43, Resistor_SMD:R_0815_2038Metric_Pad1.20x4.05mm_HandSolder, F.Cu at (-76.1, -147.1)
- added R16: R732, Resistor_SMD:R_0815_2038Metric_Pad1.20x4.05mm_HandSolder, F.Cu at (-71.3, -147.1)
- added U11: DRV8874PWPR, footprints:PWP0016J_NV, F.Cu at (44.7, 44.2)
- added U19: 7410, Package_SO:SOIC-14_3.9x8.7mm_P1.27mm, F.Cu at (-70.5, -155.6)
- added U21: DRV8874PWPR, footprints:PWP0016J_NV, F.Cu at (45.0, 80.0)
- added U22: 7410, Package_SO:SOIC-14_3.9x8.7mm_P1.27mm, F.Cu at (-129.2, -120.1)
- added U40: 7410, Package_SO:SOIC-14_3.9x8.7mm_P1.27mm, F.Cu at (-62.1, -84.6)
- added U41: DRV8874PWPR, footprints:PWP0016J_NV, F.Cu at (45.0, 151.9)
- C13, C15, C21, C33, C45: value C10u -> C100n
- C16, C18, C23, C24, C35, C36, C41, C42, C48, C6: value C22n -> C100n
- C17, C47: value C22n -> C10u
- C19, C20, C40: value C100n -> C22n
- C37: value C100n -> C10u
- C39: value C10u -> C22n
- J4: value Screw_Terminal_01x12 -> Screw_Terminal_01x02; footprint TerminalBlock_4Ucon:TerminalBlock_4Ucon_1x12_P3.50mm_Horizontal -> TerminalBlock_Phoenix:TerminalBlock_Phoenix_MKDS-1,5-2_1x02_P5.00mm_Horizontal
- R10: value R47k -> R732
- R11, R8: value R1k43 -> R47k
- R12, R9: value R732 -> R1k43
- U1: value DRV8874PWPR -> ACPL-214-500E; footprint footprints:PWP0016J_NV -> Package_SO:SOP-4_4.4x2.6mm_P1.27mm
- U10, U15, U20, U27, U35, U39: value DRV8874PWPR -> 7410; footprint footprints:PWP0016J_NV -> Package_SO:SOIC-14_3.9x8.7mm_P1.27mm
- U12, U13, U14, U17, U18, U2, U24, U25, U28, U29, U3, U30, U32, U33, U34, U37, U38, U4, U7, U8, U9: footprint Package_SO:SO-14_5.3x10.2mm_P1.27mm -> Package_SO:SOIC-14_3.9x8.7mm_P1.27mm
- U16, U36: value 7404 -> DRV8874PWPR; footprint Package_SO:SO-14_5.3x10.2mm_P1.27mm -> footprints:PWP0016J_NV
- U23, U5: value 7404 -> 7410; footprint Package_SO:SO-14_5.3x10.2mm_P1.27mm -> Package_SO:SOIC-14_3.9x8.7mm_P1.27mm
- U26: value 7410 -> DRV8874PWPR; footprint Package_SO:SO-14_5.3x10.2mm_P1.27mm -> footprints:PWP0016J_NV
- U6: value ACPL-214-500E -> DRV8874PWPR; footprint Package_SO:SOP-4_4.4x2.6mm_P1.27mm -> footprints:PWP0016J_NV
- moved C21 387.1 mm to (-136.5, -159.8)
- moved C22 387.1 mm to (-136.5, -156.4)
- moved C23 387.1 mm to (-136.5, -153.1)
- moved C24 387.1 mm to (-136.5, -149.7)
- moved R11 386.8 mm to (-122.8, -147.1)
- moved R12 386.8 mm to (-117.9, -147.1)
- moved U18 354.4 mm to (-79.0, -155.6)
- moved U17 353.0 mm to (-87.4, -155.6)
- moved C41 351.1 mm to (-136.5, -124.3)
- moved C42 351.1 mm to (-136.5, -120.9)
- moved Q4 347.1 mm to (-66.5, -147.5)
- moved U20 342.3 mm to (-62.1, -155.6)
- moved C31 336.9 mm to (-94.6, -159.8)
- moved C32 336.9 mm to (-94.6, -156.4)
- moved C33 336.9 mm to (-94.6, -153.1)
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- renumbered J3 to J1, J2 to J6, R13 to R1, R15 to R2, R16 to R3, R14 to R4, U11 to U42, U40 to U43, U21 to U44, U41 to U45
Connections:
- C10 pad 1: /sense_B -> /sense_A
- C12 pad 1: VTRACK -> (no net)
- C12 pad 2: Net-(U15-VCP) -> (no net)
- C13 pad 1: VTRACK -> IOREF
- C14 pad 1: VTRACK -> IOREF
- C15 pad 1: VTRACK -> IOREF
- C16 pad 1: Net-(U15-CPH) -> VTRACK
- C16 pad 2: Net-(U15-CPL) -> Net-(U11-VCP)
- C17 pad 1: /sense_C -> VTRACK
- C18 pad 1: /sense_A -> VTRACK
- C19 pad 1: IOREF -> Net-(U11-CPH)
- C19 pad 2: GND -> Net-(U11-CPL)
- C2 pad 1: VTRACK -> IOREF
- C20 pad 1: VTRACK -> /sense_B
- C20 pad 2: Net-(U20-VCP) -> GND
- C21 pad 1: VTRACK -> IOREF
- C22 pad 1: VTRACK -> IOREF
- C23 pad 1: Net-(U20-CPH) -> IOREF
- C23 pad 2: Net-(U20-CPL) -> GND
- C24 pad 1: /sense_D -> IOREF
- C26 pad 2: Net-(U27-VCP) -> Net-(U16-VCP)
- C29 pad 1: Net-(U27-CPH) -> Net-(U16-CPH)
- C29 pad 2: Net-(U27-CPL) -> Net-(U16-CPL)
- C3 pad 1: VTRACK -> IOREF
- C3 pad 2: Net-(U10-VCP) -> GND
- C30 pad 1: /sense_E -> /sense_C
- C32 pad 1: VTRACK -> IOREF
- C32 pad 2: Net-(U31-VCP) -> GND
- C33 pad 1: VTRACK -> IOREF
- C34 pad 1: VTRACK -> IOREF
- C35 pad 1: Net-(U31-CPH) -> IOREF
- C35 pad 2: Net-(U31-CPL) -> GND
- C36 pad 1: /sense_F -> VTRACK
- C36 pad 2: GND -> Net-(U21-VCP)
- C37 pad 1: IOREF -> VTRACK
- C38 pad 2: Net-(U35-VCP) -> GND
- C39 pad 1: VTRACK -> Net-(U21-CPH)
- C39 pad 2: GND -> Net-(U21-CPL)
- C40 pad 1: VTRACK -> /sense_D
- C41 pad 1: Net-(U35-CPH) -> IOREF
- C41 pad 2: Net-(U35-CPL) -> GND
- C42 pad 1: /sense_G -> IOREF
- C44 pad 1: VTRACK -> IOREF
- C44 pad 2: Net-(U39-VCP) -> GND
- C45 pad 1: VTRACK -> IOREF
- C46 pad 2: GND -> Net-(U26-VCP)
- C47 pad 1: Net-(U39-CPH) -> VTRACK
- C47 pad 2: Net-(U39-CPL) -> GND
- C48 pad 1: /sense_H -> VTRACK
- C5 pad 1: VTRACK -> IOREF
- C5 pad 2: Net-(U1-VCP) -> GND
- C6 pad 1: Net-(U1-CPH) -> VTRACK
- C6 pad 2: Net-(U1-CPL) -> Net-(U6-VCP)
- C9 pad 1: Net-(U10-CPH) -> Net-(U6-CPH)
- C9 pad 2: Net-(U10-CPL) -> Net-(U6-CPL)
- J4 pad 1: VTRACK -> /raw_dcc_p
- J4 pad 2: GND -> /raw_dcc_n
- R10 pad 1: IOREF -> Net-(Q2-D)
- R10 pad 2: Net-(U20-FAULT_N) -> GND
- R11 pad 1: /sense_D -> IOREF
- R11 pad 2: Net-(Q4-D) -> Net-(U16-FAULT_N)
- R12 pad 1: Net-(Q4-D) -> /sense_C
- R12 pad 2: GND -> Net-(Q3-D)
- R17 pad 2: Net-(U27-FAULT_N) -> Net-(U26-FAULT_N)
- R23 pad 2: Net-(U35-FAULT_N) -> Net-(U36-FAULT_N)
- R26 pad 2: Net-(U39-FAULT_N) -> Net-(U41-FAULT_N)
- R5 pad 2: Net-(U15-FAULT_N) -> Net-(U6-FAULT_N)
- R6 pad 1: /sense_C -> /sense_A
- R6 pad 2: Net-(Q3-D) -> Net-(Q1-D)
- R7 pad 1: Net-(Q3-D) -> Net-(Q1-D)
- R8 pad 1: /sense_A -> IOREF
- R8 pad 2: Net-(Q1-D) -> Net-(U11-FAULT_N)
- R9 pad 1: Net-(Q1-D) -> /sense_B
- R9 pad 2: GND -> Net-(Q2-D)
- U1 pad 1: Net-(U1-EN_IN1) -> /raw_dcc_p
- U1 pad 2: Net-(U1-PH_IN2) -> GND
- U1 pad 3: IOREF -> /dcc_p
- U1 pad 4: Net-(U1-FAULT_N) -> IOREF
- U10 pad 1: Net-(U10-EN_IN1) -> Net-(U10-Pad1)
- U10 pad 10: /out2_B -> unconnected-(U10-Pad10)
- U10 pad 11: VTRACK -> unconnected-(U10-Pad11)
- U10 pad 12: Net-(U10-VCP) -> Net-(U11-EN_IN1)
- U10 pad 13: Net-(U10-CPH) -> Net-(U10-Pad13)
- U10 pad 14: Net-(U10-CPL) -> IOREF
- U10 pad 2: Net-(U10-PH_IN2) -> Net-(U10-Pad2)
- U10 pad 3: IOREF -> Net-(U10-Pad3)
- U10 pad 4: Net-(U10-FAULT_N) -> Net-(U10-Pad4)
- U10 pad 5: IOREF -> Net-(U10-Pad5)
- U10 pad 6: /sense_B -> Net-(U11-PH_IN2)
- U10 pad 8: /out1_B -> unconnected-(U10-Pad8)
- U10 pad 9: GND -> unconnected-(U10-Pad9)
- U12 pad 1: /dcc_n -> /dcc_en_C
- U12 pad 10: Net-(U12-Pad10) -> /dcc_p
- U12 pad 11: Net-(U12-Pad11) -> /dcc_p
- U12 pad 13: /dir_C -> /dcc_en_C
- U12 pad 3: /dcc_p -> /dir_C
- U12 pad 4: /dcc_en_C -> /dir_C
- U12 pad 5: Net-(U12-Pad11) -> /dir_C
- U12 pad 9: /pwm_C -> /dcc_p
- U13 pad 1: /dcc_p -> Net-(U12-Pad8)
- U13 pad 10: Net-(U12-Pad10) -> Net-(U12-Pad12)
- U13 pad 11: /dir_C -> Net-(U12-Pad6)
- U13 pad 3: /dcc_n -> /dcc_p
- U13 pad 5: Net-(U12-Pad11) -> Net-(U12-Pad6)
- U14 pad 1: Net-(U12-Pad12) -> /dcc_p
- U14 pad 10: (no net) -> Net-(U12-Pad12)
- U14 pad 11: (no net) -> /dir_C
- U14 pad 12: Net-(U15-EN_IN1) -> Net-(U14-Pad12)
- U14 pad 13: Net-(U12-Pad8) -> /dir_C
- U14 pad 2: Net-(U12-Pad6) -> /dcc_en_C
- U14 pad 3: Net-(U13-Pad12) -> Net-(U12-Pad8)
- U14 pad 4: Net-(U13-Pad6) -> /dcc_en_C
- U14 pad 5: Net-(U13-Pad8) -> Net-(U12-Pad6)
- U14 pad 6: Net-(U15-PH_IN2) -> Net-(U14-Pad6)
- U14 pad 8: (no net) -> Net-(U14-Pad8)
- U14 pad 9: (no net) -> /pwm_C
- U15 pad 1: Net-(U15-EN_IN1) -> Net-(U13-Pad12)
- U15 pad 10: /out2_C -> unconnected-(U15-Pad10)
- U15 pad 11: VTRACK -> unconnected-(U15-Pad11)
- U15 pad 12: Net-(U15-VCP) -> Net-(U16-EN_IN1)
- U15 pad 13: Net-(U15-CPH) -> Net-(U13-Pad8)
- U15 pad 14: Net-(U15-CPL) -> IOREF
- U15 pad 2: Net-(U15-PH_IN2) -> Net-(U13-Pad6)
- U15 pad 3: IOREF -> Net-(U14-Pad12)
- U15 pad 4: Net-(U15-FAULT_N) -> Net-(U14-Pad6)
- U15 pad 5: IOREF -> Net-(U14-Pad8)
- U15 pad 6: /sense_C -> Net-(U16-PH_IN2)
- U15 pad 8: /out1_C -> unconnected-(U15-Pad8)
- U15 pad 9: GND -> unconnected-(U15-Pad9)
- U16 pad 1: /dcc_en_D -> Net-(U16-EN_IN1)
- U16 pad 10: (no net) -> /out2_C
- U16 pad 11: (no net) -> VTRACK
- U16 pad 12: (no net) -> Net-(U16-VCP)
- U16 pad 13: (no net) -> Net-(U16-CPH)
- U16 pad 14: IOREF -> Net-(U16-CPL)
- U16 pad 2: Net-(U16-Pad2) -> Net-(U16-PH_IN2)
- U16 pad 3: /dir_D -> IOREF
- U16 pad 4: Net-(U16-Pad4) -> Net-(U16-FAULT_N)
- U16 pad 5: /dcc_p -> IOREF
- U16 pad 6: /dcc_n -> /sense_C
- U16 pad 8: (no net) -> /out1_C
- U16 pad 9: (no net) -> GND
- U17 pad 1: /dcc_n -> /dcc_en_D
- U17 pad 10: Net-(U16-Pad2) -> /dcc_p
- U17 pad 11: Net-(U16-Pad4) -> /dcc_p
- U17 pad 13: /dir_D -> /dcc_en_D
- U17 pad 3: /dcc_p -> /dir_D
- U17 pad 4: /dcc_en_D -> /dir_D
- U17 pad 5: Net-(U16-Pad4) -> /dir_D
- U17 pad 9: /pwm_D -> /dcc_p
- U18 pad 1: /dcc_p -> Net-(U17-Pad8)
- U18 pad 10: Net-(U16-Pad2) -> Net-(U17-Pad12)
- U18 pad 11: /dir_D -> Net-(U17-Pad6)
- U18 pad 3: /dcc_n -> /dcc_p
- U18 pad 5: Net-(U16-Pad4) -> Net-(U17-Pad6)
- U2 pad 1: /dcc_n -> /dcc_en_A
- U2 pad 10: Net-(U2-Pad10) -> /dcc_p
- U2 pad 11: Net-(U2-Pad11) -> /dcc_p
- U2 pad 13: /dir_A -> /dcc_en_A
- U2 pad 3: /dcc_p -> /dir_A
- U2 pad 4: /dcc_en_A -> /dir_A
- U2 pad 5: Net-(U2-Pad11) -> /dir_A
- U2 pad 9: /pwm_A -> /dcc_p
- U20 pad 1: Net-(U20-EN_IN1) -> Net-(U18-Pad12)
- U20 pad 10: /out2_D -> unconnected-(U20-Pad10)
- U20 pad 11: VTRACK -> unconnected-(U20-Pad11)
- U20 pad 12: Net-(U20-VCP) -> Net-(U21-EN_IN1)
- U20 pad 13: Net-(U20-CPH) -> Net-(U18-Pad8)
- U20 pad 14: Net-(U20-CPL) -> IOREF
- U20 pad 2: Net-(U20-PH_IN2) -> Net-(U18-Pad6)
- U20 pad 3: IOREF -> Net-(U19-Pad12)
- U20 pad 4: Net-(U20-FAULT_N) -> Net-(U19-Pad6)
- U20 pad 5: IOREF -> Net-(U19-Pad8)
- U20 pad 6: /sense_D -> Net-(U21-PH_IN2)
- U20 pad 8: /out1_D -> unconnected-(U20-Pad8)
- U20 pad 9: GND -> unconnected-(U20-Pad9)
- U23 pad 1: /dcc_en_E -> Net-(U22-Pad8)
- U23 pad 10: Net-(U23-Pad10) -> Net-(U22-Pad12)
- U23 pad 11: /dcc_en_G -> Net-(U22-Pad6)
- U23 pad 13: /dir_G -> /dir_E
- U23 pad 2: Net-(U23-Pad2) -> /dcc_en_E
- U23 pad 3: /dir_E -> /dcc_p
- U23 pad 4: Net-(U23-Pad4) -> /dcc_en_E
- U23 pad 5: /dcc_en_F -> Net-(U22-Pad6)
- U23 pad 9: /dir_F -> /pwm_E
- U24 pad 1: /dcc_n -> /dcc_p
- U24 pad 10: Net-(U23-Pad2) -> Net-(U22-Pad12)
- U24 pad 11: Net-(U23-Pad4) -> /dir_E
- U24 pad 3: /dcc_p -> Net-(U22-Pad8)
- U24 pad 5: Net-(U23-Pad4) -> Net-(U22-Pad6)
- U25 pad 1: /dcc_p -> Net-(U23-Pad12)
- U25 pad 10: Net-(U23-Pad2) -> unconnected-(U25-Pad10)
- U25 pad 11: /dir_E -> unconnected-(U25-Pad11)
- U25 pad 12: Net-(U25-Pad12) -> Net-(U26-EN_IN1)
- U25 pad 13: /dir_E -> Net-(U23-Pad8)
- U25 pad 2: /dcc_en_E -> Net-(U23-Pad6)
- U25 pad 3: /dcc_n -> Net-(U24-Pad12)
- U25 pad 4: /dcc_en_E -> Net-(U24-Pad6)
- U25 pad 5: Net-(U23-Pad4) -> Net-(U24-Pad8)
- U25 pad 6: Net-(U25-Pad6) -> Net-(U26-PH_IN2)
- U25 pad 8: Net-(U25-Pad8) -> unconnected-(U25-Pad8)
- U25 pad 9: /pwm_E -> unconnected-(U25-Pad9)
- U26 pad 1: Net-(U24-Pad12) -> Net-(U26-EN_IN1)
- U26 pad 10: Net-(U26-Pad10) -> /out2_E
- U26 pad 11: Net-(U26-Pad11) -> VTRACK
- U26 pad 12: Net-(U27-EN_IN1) -> Net-(U26-VCP)
- U26 pad 13: Net-(U24-Pad8) -> Net-(U26-CPH)
- U26 pad 14: IOREF -> Net-(U26-CPL)
- U26 pad 2: Net-(U24-Pad6) -> Net-(U26-PH_IN2)
- U26 pad 3: Net-(U25-Pad12) -> IOREF
- U26 pad 4: Net-(U25-Pad6) -> Net-(U26-FAULT_N)
- U26 pad 5: Net-(U25-Pad8) -> IOREF
- U26 pad 6: Net-(U27-PH_IN2) -> /sense_E
- U26 pad 8: Net-(U39-EN_IN1) -> /out1_E
- U26 pad 9: Net-(U26-Pad9) -> GND
- U27 pad 1: Net-(U27-EN_IN1) -> /dcc_en_F
- U27 pad 10: /out2_E -> /dcc_p
- U27 pad 11: VTRACK -> /dcc_p
- U27 pad 12: Net-(U27-VCP) -> Net-(U27-Pad12)
- U27 pad 13: Net-(U27-CPH) -> /dcc_en_F
- U27 pad 14: Net-(U27-CPL) -> IOREF
- U27 pad 2: Net-(U27-PH_IN2) -> /dcc_en_F
- U27 pad 3: IOREF -> /dir_F
- U27 pad 4: Net-(U27-FAULT_N) -> /dir_F
- U27 pad 5: IOREF -> /dir_F
- U27 pad 6: /sense_E -> Net-(U27-Pad6)
- U27 pad 8: /out1_E -> Net-(U27-Pad8)
- U27 pad 9: GND -> /dcc_p
- U28 pad 1: /dcc_n -> Net-(U27-Pad8)
- U28 pad 10: Net-(U23-Pad6) -> Net-(U27-Pad12)
- U28 pad 11: Net-(U23-Pad8) -> Net-(U27-Pad6)
- U28 pad 5: Net-(U23-Pad8) -> Net-(U27-Pad6)
- U29 pad 10: Net-(U23-Pad6) -> Net-(U27-Pad12)
- U29 pad 3: /dcc_n -> Net-(U27-Pad8)
- U29 pad 5: Net-(U23-Pad8) -> Net-(U27-Pad6)
- U3 pad 1: Net-(U2-Pad12) -> Net-(U2-Pad8)
- U3 pad 10: Net-(U17-Pad6) -> Net-(U2-Pad12)
- U3 pad 11: Net-(U17-Pad8) -> Net-(U2-Pad6)
- U3 pad 12: Net-(U1-EN_IN1) -> Net-(U3-Pad12)
- U3 pad 13: Net-(U2-Pad8) -> /dir_A
- U3 pad 2: Net-(U2-Pad6) -> /dcc_en_A
- U3 pad 3: Net-(U3-Pad3) -> /dcc_p
- U3 pad 4: Net-(U3-Pad4) -> /dcc_en_A
- U3 pad 5: Net-(U3-Pad5) -> Net-(U2-Pad6)
- U3 pad 6: Net-(U1-PH_IN2) -> Net-(U3-Pad6)
- U3 pad 8: Net-(U20-EN_IN1) -> Net-(U3-Pad8)
- U3 pad 9: Net-(U17-Pad12) -> /pwm_A
- U30 pad 10: Net-(U30-Pad10) -> unconnected-(U30-Pad10)
- U30 pad 11: Net-(U30-Pad11) -> unconnected-(U30-Pad11)
- U30 pad 8: Net-(U39-PH_IN2) -> unconnected-(U30-Pad8)
- U30 pad 9: Net-(U30-Pad9) -> unconnected-(U30-Pad9)
- U32 pad 1: /dcc_n -> /dcc_en_G
- U32 pad 10: Net-(U23-Pad10) -> /dcc_p
- U32 pad 11: Net-(U23-Pad12) -> /dcc_p
- U32 pad 13: /dir_G -> /dcc_en_G
- U32 pad 3: /dcc_p -> /dir_G
- U32 pad 4: /dcc_en_G -> /dir_G
- U32 pad 5: Net-(U23-Pad12) -> /dir_G
- U32 pad 9: /pwm_G -> /dcc_p
- U33 pad 1: /dcc_p -> Net-(U32-Pad8)
- U33 pad 10: Net-(U23-Pad10) -> Net-(U32-Pad12)
- U33 pad 11: /dir_G -> Net-(U32-Pad6)
- U33 pad 3: /dcc_n -> /dcc_p
- U33 pad 5: Net-(U23-Pad12) -> Net-(U32-Pad6)
- U34 pad 1: Net-(U32-Pad12) -> /dcc_p
- U34 pad 10: (no net) -> Net-(U32-Pad12)
- U34 pad 11: (no net) -> /dir_G
- U34 pad 12: Net-(U35-EN_IN1) -> Net-(U34-Pad12)
- U34 pad 13: Net-(U32-Pad8) -> /dir_G
- U34 pad 2: Net-(U32-Pad6) -> /dcc_en_G
- U34 pad 3: Net-(U33-Pad12) -> Net-(U32-Pad8)
- U34 pad 4: Net-(U33-Pad6) -> /dcc_en_G
- U34 pad 5: Net-(U33-Pad8) -> Net-(U32-Pad6)
- U34 pad 6: Net-(U35-PH_IN2) -> Net-(U34-Pad6)
- U34 pad 8: (no net) -> Net-(U34-Pad8)
- U34 pad 9: (no net) -> /pwm_G
- U35 pad 1: Net-(U35-EN_IN1) -> Net-(U33-Pad12)
- U35 pad 10: /out2_G -> unconnected-(U35-Pad10)
- U35 pad 11: VTRACK -> unconnected-(U35-Pad11)
- U35 pad 12: Net-(U35-VCP) -> Net-(U36-EN_IN1)
- U35 pad 13: Net-(U35-CPH) -> Net-(U33-Pad8)
- U35 pad 14: Net-(U35-CPL) -> IOREF
- U35 pad 2: Net-(U35-PH_IN2) -> Net-(U33-Pad6)
- U35 pad 3: IOREF -> Net-(U34-Pad12)
- U35 pad 4: Net-(U35-FAULT_N) -> Net-(U34-Pad6)
- U35 pad 5: IOREF -> Net-(U34-Pad8)
- U35 pad 6: /sense_G -> Net-(U36-PH_IN2)
- U35 pad 8: /out1_G -> unconnected-(U35-Pad8)
- U35 pad 9: GND -> unconnected-(U35-Pad9)
- U36 pad 1: /dcc_en_H -> Net-(U36-EN_IN1)
- U36 pad 10: (no net) -> /out2_G
- U36 pad 11: (no net) -> VTRACK
- U36 pad 12: (no net) -> Net-(U36-VCP)
- U36 pad 13: (no net) -> Net-(U36-CPH)
- U36 pad 14: IOREF -> Net-(U36-CPL)
- U36 pad 2: Net-(U36-Pad2) -> Net-(U36-PH_IN2)
- U36 pad 3: /dir_H -> IOREF
- U36 pad 4: Net-(U36-Pad4) -> Net-(U36-FAULT_N)
- U36 pad 5: (no net) -> IOREF
- U36 pad 6: (no net) -> /sense_G
- U36 pad 8: (no net) -> /out1_G
- U36 pad 9: (no net) -> GND
- U37 pad 1: /dcc_n -> /dcc_en_H
- U37 pad 10: Net-(U36-Pad2) -> /dcc_p
- U37 pad 11: Net-(U36-Pad4) -> /dcc_p
- U37 pad 12: Net-(U26-Pad9) -> Net-(U37-Pad12)
- U37 pad 13: /dir_H -> /dcc_en_H
- U37 pad 3: /dcc_p -> /dir_H
- U37 pad 4: /dcc_en_H -> /dir_H
- U37 pad 5: Net-(U36-Pad4) -> /dir_H
- U37 pad 6: Net-(U26-Pad10) -> Net-(U37-Pad6)
- U37 pad 8: Net-(U26-Pad11) -> Net-(U37-Pad8)
- U37 pad 9: /pwm_H -> /dcc_p
- U38 pad 1: /dcc_p -> Net-(U37-Pad8)
- U38 pad 10: Net-(U36-Pad2) -> Net-(U37-Pad12)
- U38 pad 11: /dir_H -> Net-(U37-Pad6)
- U38 pad 12: Net-(U30-Pad9) -> Net-(U38-Pad12)
- U38 pad 3: /dcc_n -> /dcc_p
- U38 pad 5: Net-(U36-Pad4) -> Net-(U37-Pad6)
- U38 pad 6: Net-(U30-Pad10) -> Net-(U38-Pad6)
- U38 pad 8: Net-(U30-Pad11) -> Net-(U38-Pad8)
- U39 pad 1: Net-(U39-EN_IN1) -> /dcc_p
- U39 pad 10: /out2_H -> Net-(U37-Pad12)
- U39 pad 11: VTRACK -> /dir_H
- U39 pad 12: Net-(U39-VCP) -> Net-(U39-Pad12)
- U39 pad 13: Net-(U39-CPH) -> /dir_H
- U39 pad 14: Net-(U39-CPL) -> IOREF
- U39 pad 2: Net-(U39-PH_IN2) -> /dcc_en_H
- U39 pad 3: IOREF -> Net-(U37-Pad8)
- U39 pad 4: Net-(U39-FAULT_N) -> /dcc_en_H
- U39 pad 5: IOREF -> Net-(U37-Pad6)
- U39 pad 6: /sense_H -> Net-(U39-Pad6)
- U39 pad 8: /out1_H -> Net-(U39-Pad8)
- U39 pad 9: GND -> /pwm_H
- U4 pad 10: Net-(U2-Pad10) -> Net-(U2-Pad12)
- U4 pad 12: Net-(U3-Pad3) -> Net-(U4-Pad12)
- U4 pad 3: /dcc_n -> Net-(U2-Pad8)
- U4 pad 5: Net-(U2-Pad11) -> Net-(U2-Pad6)
- U4 pad 6: Net-(U3-Pad4) -> Net-(U4-Pad6)
- U4 pad 8: Net-(U3-Pad5) -> Net-(U4-Pad8)
- U5 pad 1: /dcc_en_A -> Net-(U3-Pad12)
- U5 pad 10: Net-(U12-Pad10) -> unconnected-(U5-Pad10)
- U5 pad 11: /dcc_en_C -> unconnected-(U5-Pad11)
- U5 pad 12: Net-(U12-Pad11) -> Net-(U6-EN_IN1)
- U5 pad 13: /dir_C -> Net-(U3-Pad8)
- U5 pad 2: Net-(U2-Pad10) -> Net-(U3-Pad6)
- U5 pad 3: /dir_A -> Net-(U4-Pad12)
- U5 pad 4: Net-(U2-Pad11) -> Net-(U4-Pad6)
- U5 pad 5: /dcc_en_B -> Net-(U4-Pad8)
- U5 pad 6: Net-(U5-Pad6) -> Net-(U6-PH_IN2)
- U5 pad 8: Net-(U5-Pad8) -> unconnected-(U5-Pad8)
- U5 pad 9: /dir_B -> unconnected-(U5-Pad9)
- U6 pad 1: /raw_dcc_p -> Net-(U6-EN_IN1)
- U6 pad 2: GND -> Net-(U6-PH_IN2)
- U6 pad 3: /dcc_p -> IOREF
- U6 pad 4: IOREF -> Net-(U6-FAULT_N)
- U7 pad 1: /dcc_n -> /dcc_en_B
- U7 pad 10: Net-(U5-Pad6) -> /dcc_p
- U7 pad 11: Net-(U5-Pad8) -> /dcc_p
- U7 pad 13: /dir_B -> /dcc_en_B
- U7 pad 3: /dcc_p -> /dir_B
- U7 pad 4: /dcc_en_B -> /dir_B
- U7 pad 5: Net-(U5-Pad8) -> /dir_B
- U7 pad 9: /pwm_B -> /dcc_p
- U8 pad 1: /dcc_p -> Net-(U7-Pad8)
- U8 pad 10: Net-(U5-Pad6) -> Net-(U7-Pad12)
- U8 pad 11: /dir_B -> Net-(U7-Pad6)
- U8 pad 12: Net-(U8-Pad12) -> Net-(U10-Pad1)
- U8 pad 3: /dcc_n -> /dcc_p
- U8 pad 5: Net-(U5-Pad8) -> Net-(U7-Pad6)
- U8 pad 6: Net-(U8-Pad6) -> Net-(U10-Pad2)
- U8 pad 8: Net-(U8-Pad8) -> Net-(U10-Pad13)
- U9 pad 1: Net-(U7-Pad12) -> /dcc_p
- U9 pad 10: Net-(U18-Pad6) -> Net-(U7-Pad12)
- U9 pad 11: Net-(U18-Pad8) -> /dir_B
- U9 pad 12: Net-(U10-EN_IN1) -> Net-(U10-Pad3)
- U9 pad 13: Net-(U7-Pad8) -> /dir_B
- U9 pad 2: Net-(U7-Pad6) -> /dcc_en_B
- U9 pad 3: Net-(U8-Pad12) -> Net-(U7-Pad8)
- U9 pad 4: Net-(U8-Pad6) -> /dcc_en_B
- U9 pad 5: Net-(U8-Pad8) -> Net-(U7-Pad6)
- U9 pad 6: Net-(U10-PH_IN2) -> Net-(U10-Pad4)
- U9 pad 8: Net-(U20-PH_IN2) -> Net-(U10-Pad5)
- U9 pad 9: Net-(U18-Pad12) -> /pwm_B
Routing:
- net GND: track 0.00 -> 816.1 mm, vias 0 -> 25
- net IOREF: track 0.00 -> 316.1 mm, vias 0 -> 17
- net VTRACK: track 0.00 -> 235.2 mm, vias 0 -> 8
- net +5V: track 0.00 -> 181.3 mm, vias 0 -> 3
- net +3.3V: track 0.00 -> 137.5 mm
- net /raw_dcc_p: track 0.00 -> 126.3 mm
- net /raw_dcc_n: track 0.00 -> 125.2 mm
- net VIN: track 0.00 -> 103.9 mm, vias 0 -> 2
- net /sense_A: track 0.00 -> 49.4 mm
- net /sck_2: track 0.00 -> 46.9 mm
- net /sck_1: track 0.00 -> 46.6 mm
- net /out2_H: track 0.00 -> 39.4 mm
- net /out1_A: track 0.00 -> 39.2 mm
- net /out2_A: track 0.00 -> 38.9 mm
- net /cs_1: track 0.00 -> 35.9 mm
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- added copper zone on B.Cu, net GND
- added copper zone on F.Cu, net GND
Other:
- board size 213.4 x 137.2 mm -> 155 x 155 mm
- board text added: "DCC+"
- board text added: "DCC-"
- board text added: "GND"
- board text added: "V_TRACK"
