File: hardware/Uno_R4_LCC_Shield/Uno_R4_LCC_Shield.kicad_sch (KiCad schematic)
At the start: 4 parts, among them U1 MCP2515-xSO, U2 MCP2562-E-SN, Y1 16.0 MHz, 22pF

Commit message: Better Solder Jumpers, Better Pizza
Parts:
- removed U1: MCP2515-xSO, Package_SO:SOIC-18W_7.5x11.6mm_P1.27mm, symbol Interface_CAN_LIN:MCP2515-xSO
- removed U2: MCP2562-E-SN, Package_SO:SOIC-8_3.9x4.9mm_P1.27mm, symbol Interface_CAN_LIN:MCP2562-E-SN
- removed Y1: 16.0 MHz, 22pF, Crystal:Crystal_HC49-U-3Pin_Vertical, symbol Device:Resonator_Small
- added J1: A00-216-262-450, A00_216_262_450:EDAC_A00-216-262-450, symbol A00-216-262-450:A00-216-262-450
- added J2: 54-00166, 54-00166:TENSILITY_54-00166, symbol 54-00166:54-00166
- added J3: Screw_Terminal_01x02, TerminalBlock_Phoenix:TerminalBlock_Phoenix_MKDS-1,5-2_1x02_P5.00mm_Horizontal, symbol Connector:Screw_Terminal_01x02
- added JP1, JP2, JP3, JP4: SolderJumper_2_Open, Jumper:SolderJumper-2_P1.3mm_Open_RoundedPad1.0x1.5mm, symbol Jumper:SolderJumper_2_Open
- added JP5, JP6: SolderJumper_3_Bridged12, Jumper:SolderJumper-3_P1.3mm_Bridged12_RoundedPad1.0x1.5mm, symbol Jumper:SolderJumper_3_Bridged12
- added SW1: SW_Push, Button_Switch_THT:SW_PUSH_6mm_H4.3mm, symbol Switch:SW_Push
- added U1: ACPL-214-500E, Package_SO:SOP-4_4.4x2.6mm_P1.27mm, symbol Isolator:ACPL-214-500E
- A1: footprint Module:Arduino_UNO_R3 -> Uno_Shield:Uno_Shield
Connections:
- net +5V: now also A1.5 (+5V)
- net GND: now also A1.29 (GND), A1.6 (GND), A1.7 (GND), J1.11 (3), J1.3, J2.B, J2.C, JP4.2 (B), SW1.1, U1.2
- net IOREF: now also U1.4
- net can_h: now also J1.1, J1.9 (1)
- net can_l: now also J1.10 (2), J1.2
- net ~{reset}: now also A1.3 (~{RESET}), SW1.2
- net dcc_p: now reaches A1.17 (D2)
- net dcc_p: now also U1.3
- net pwm_A: now reaches A1.18 (D3)
- net at A1.19 (D4): now also JP6.1 (A)
- net at A1.20 (D5): now also JP5.1 (A)
- net dir_A: now reaches A1.21 (D6)
- net dcc_en_A: now reaches A1.22 (D7)
- net at A1.25 (D10): now also JP6.3 (B)
- net at A1.28 (D13): now also JP5.3 (B)
- net +3.3V: now reaches A1.4 (3V3)
- net VIN: now reaches A1.8 (VIN)
- net VIN: now also JP1.2 (B)
- net sense_A: now reaches A1.9 (A0)
- new net VTRACK: J2.A, JP1.1 (A)
- new net can_rx: JP5.2 (C)
- new net can_shield: J1.14 (6), J1.6, J1.M1 (SHIELD), J1.M2 (SHIELD), JP4.1 (A)
- new net can_tx: JP6.2 (C)
- new net out1_A: J3.2 (Pin_2), JP3.2 (B)
- new net out2_A: J3.1 (Pin_1), JP2.2 (B)
- new net pwr_n: J1.15 (7), J1.7
- new net pwr_p: J1.16 (8), J1.8
- new net raw_dcc_n: J1.12 (4), J1.4, JP2.1 (A)
- new net raw_dcc_p: J1.13 (5), J1.5, JP3.1 (A), U1.1
- no-connect marks 8 -> 14
Other:
- added sheet Block Driver A (block_driver.kicad_sch)
- added sheet CAN Interface (can_interface.kicad_sch)
- moved on the sheet: A1

Commit message: Update to hardware v2 and cleanup
Parts:
- added C8, C9: C100n, Capacitor_SMD:C_0402_1005Metric_Pad0.74x0.62mm_HandSolder, symbol Device:C
- added U4: ACPL-214-500E, Package_SO:SOP-4_4.4x2.6mm_P1.27mm, symbol Isolator:ACPL-214-500E
Connections:
- net GND: now also C8.2, C9.2, U4.2
- net IOREF: now also C8.1, C9.1, U4.4
- net raw_dcc_n: now also U4.1
- new net dcc_n: U4.3
Other:
- sheet Block Driver A ports: added DCC_n; removed none

Commit message: Small tweaks to pinout on Uno R4 Shield and additional cleanup
Connections:
- net dcc_p: now also A1.23 (D8); no longer A1.17 (D2)
- new net nFault_A: A1.17 (D2)
- no-connect marks 14 -> 13
Other:
- sheet Block Driver A ports: added FAULT_N; removed none
Changed lines of the file:
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@@
 		(at 72.39 81.28)
 	)
-	(no_connect
-		(at 72.39 73.66)
-	)
 	(wire
 		(pts
@@
 	(wire
 		(pts
+			(xy 153.67 62.23) (xy 154.94 62.23)
+		)
+		(stroke
+			(width 0)
+			(type default)
+		)
+	)
+	(wire
+		(pts
 			(xy 107.95 135.89) (xy 107.95 142.24)
 		)
@@
 		)
 	)
-	(label "dcc_p"
-		(at 72.39 58.42 180)
-		(fields_autoplaced yes)
-		(effects
-			(font
-				(size 1.27 1.27)
-			)
-			(justify right bottom)
-		)
-	)
 	(label "sense_A"
 		(at 97.79 68.58 0)
@@
 		)
 	)
+	(label "nFault_A"
+		(at 72.39 58.42 180)
+		(fields_autoplaced yes)
+		(effects
+			(font
+				(size 1.27 1.27)
+			)
+			(justify right bottom)
+		)
+	)
 	(label "can_tx"
 		(at 33.02 63.5 180)
@@
 		)
 	)
+	(label "nFault_A"
+		(at 154.94 62.23 0)
+		(fields_autoplaced yes)
+		(effects
+			(font
+				(size 1.27 1.27)
+			)
+			(justify left bottom)
+		)
+	)
 	(label "~{reset}"
 		(at 219.71 129.54 0)
@@
 		)
 	)
+	(label "dcc_p"
+		(at 72.39 73.66 180)
+		(fields_autoplaced yes)
+		(effects
+			(font
+				(size 1.27 1.27)
+			)
+			(justify right bottom)
+		)
+	)
 	(label "raw_dcc_p"
 		(at 161.29 125.73 180)
@@
 			)
 		)
+		(pin "FAULT_N" output
+			(at 153.67 62.23 0)
+			(effects
+				(font
+					(size 1.27 1.27)
+				)
+				(justify right)
+			)
+		)
