File: hardware/Uno_R4_LCC_Shield/block_driver.kicad_sch (KiCad schematic)
At the start: 18 parts, among them U2 7410, U3 7410, U4 7410, U5 7410, U6 DRV8874PWPR

Commit message: Update to hardware v2 and cleanup
Parts:
- removed C10, C9: C22n, Capacitor_SMD:C_0402_1005Metric_Pad0.74x0.62mm_HandSolder, symbol Device:C
- removed C8: C100n, Capacitor_SMD:C_0402_1005Metric_Pad0.74x0.62mm_HandSolder, symbol Device:C
- removed R3: R732, Resistor_SMD:R_01005_0402Metric_Pad0.57x0.30mm_HandSolder, symbol Device:R
- removed U2, U3, U4, U5: 7410, Package_SO:SOIC-14_3.9x8.7mm_P1.27mm, symbol 74xx_IEEE:7410
- removed U6: DRV8874PWPR, ul_DRV8874PWPR:PWP0016J_NV, symbol DRV8874:DRV8874PWPR
- added U2: SN74HC253DR, Package_SO:SO-16_3.9x9.9mm_P1.27mm, symbol SN74HC253DR:SN74HC253DR
- added U3: DRV8874PWPR, DRV8874PWPR:PWP0016J_NV, symbol DRV8874:DRV8874PWPR
- C4: value C100n -> C10u; footprint Capacitor_SMD:C_0402_1005Metric_Pad0.74x0.62mm_HandSolder -> Capacitor_SMD:C_1206_3216Metric_Pad1.33x1.80mm_HandSolder
- C6: value C100n -> C22n
- C7: value C10u -> C22n; footprint Capacitor_SMD:C_1206_3216Metric_Pad1.33x1.80mm_HandSolder -> Capacitor_SMD:C_0402_1005Metric_Pad0.74x0.62mm_HandSolder
- R2: value R1k43 -> R2k
Connections:
- net DCC_EN: now also U2.2 (B)
- net DCC_p: now also U2.13 (2C3), U2.4 (1C2)
- net GND: now also R2.2, U2.1 (*1OE), U2.10 (2C0), U2.15 (*2OE), U2.5 (1C1), U2.8 (GND), U3.15 (GND), U3.17 (PAD), U3.7 (IMODE), U3.9 (PGND); no longer C3.2
- net IOREF: now also U2.16 (VCC), U3.16 (PMODE), U3.3 (SLEEP_N), U3.5 (VREF); no longer C3.1, C4.1, C5.1
- net I_SENSE: now also C7.1, U3.6 (IPROPI)
- net OUT1: now also U3.8 (OUT1)
- net OUT2: now also U3.10 (OUT2)
- net PWM: now also U2.11 (2C1), U2.6 (1C0)
- net REVERSE: now also U2.14 (A)
- net VTRACK: now also C3.1, C4.1, C5.1, U3.11 (VM); no longer C6.1, C7.1
- net at R1.2: now also U3.4 (FAULT_N)
- net at C6.2: now also U3.14 (CPL)
- new net: U2.7 (1Y), U3.1 (EN_IN1)
- new net: U2.9 (2Y), U3.2 (PH_IN2)
- new net: C3.2, U3.12 (VCP)
- new net: C6.1, U3.13 (CPH)
- new net DCC_n: U2.12 (2C2), U2.3 (1C3)
- no-connect marks 6 -> 0

Commit message: Small tweaks to pinout on Uno R4 Shield and additional cleanup
Connections:
- net FAULT_N: now reaches R1.2, U3.4 (FAULT_N)
Changed lines of the file:
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@@
+	)
+	(junction
+		(at 139.7 99.06)
+		(diameter 0)
+		(color 0 0 0 0)
 	)
 	(junction
@@
 	(wire
 		(pts
+			(xy 123.19 99.06) (xy 139.7 99.06)
+		)
+		(stroke
+			(width 0)
+			(type default)
+		)
+	)
+	(wire
+		(pts
 			(xy 118.11 83.82) (xy 111.76 83.82)
 		)
@@
 		)
 	)
+	(hierarchical_label "FAULT_N"
+		(shape output)
+		(at 123.19 99.06 180)
+		(fields_autoplaced yes)
+		(effects
+			(font
+				(size 1.27 1.27)
+			)
+			(justify right)
+		)
+	)
