File: hardware/LCC_Booster/block_driver.kicad_sch (KiCad schematic)
At the start: 13 parts, among them U5 SN74HC253DR, U6 DRV8874PWPR

Commit message: Version 5 of PCB
Parts:
- C15, C16, C17: footprint Capacitor_SMD:C_0402_1005Metric_Pad0.74x0.62mm_HandSolder -> Capacitor_SMD:C_0805_2012Metric_Pad1.18x1.45mm_HandSolder; Manufacturer Part Number CL05B104K05NNNC -> CL21B104KACNFNC
- C19: footprint Capacitor_SMD:C_0402_1005Metric_Pad0.74x0.62mm_HandSolder -> Capacitor_SMD:C_0805_2012Metric_Pad1.18x1.45mm_HandSolder; Manufacturer Part Number CL05B104KB5NFNC -> CL21B104KBFXPJE
- C20, C21: footprint Capacitor_SMD:C_0402_1005Metric_Pad0.74x0.62mm_HandSolder -> Capacitor_SMD:C_0805_2012Metric_Pad1.18x1.45mm_HandSolder; Manufacturer Part Number CL05B223KB5NNNC -> CL21B223JBANNNC
- R8: footprint Resistor_SMD:R_0402_1005Metric_Pad0.72x0.64mm_HandSolder -> Resistor_SMD:R_0805_2012Metric_Pad1.20x1.40mm_HandSolder; Manufacturer Part Number AC0402FR-071K43L -> RC0805FR-071K43L
- R9: footprint Resistor_SMD:R_0402_1005Metric_Pad0.72x0.64mm_HandSolder -> Resistor_SMD:R_0805_2012Metric_Pad1.20x1.40mm_HandSolder
Changed lines of the file:
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@@
 	(title_block
 		(title "Arduino Nano LCC Booster")
-		(date "2024-09-10")
-		(rev "4")
+		(date "2024-11-16")
+		(rev "5")
 		(company "TMRC")
 		(comment 1 "Noah Paladino")
@@
 			)
 		)
-		(property "Footprint" "Resistor_SMD:R_0402_1005Metric_Pad0.72x0.64mm_HandSolder"
+		(property "Footprint" "Resistor_SMD:R_0805_2012Metric_Pad1.20x1.40mm_HandSolder"
 			(at 198.882 132.08 90)
 			(effects
@@
 			)
 		)
-		(property "Manufacturer Part Number" "AC0402FR-071K43L"
+		(property "Manufacturer Part Number" "RC0805FR-071K43L"
 			(at 200.66 132.08 0)
 			(effects
@@
 			)
 		)
-		(property "Footprint" "Capacitor_SMD:C_0402_1005Metric_Pad0.74x0.62mm_HandSolder"
+		(property "Footprint" "Capacitor_SMD:C_0805_2012Metric_Pad1.18x1.45mm_HandSolder"
 			(at 153.3652 106.68 0)
 			(effects
@@
 			)
 		)
-		(property "Manufacturer Part Number" "CL05B104K05NNNC"
+		(property "Manufacturer Part Number" "CL21B104KACNFNC"
 			(at 152.4 102.87 0)
 			(effects
@@
 			)
 		)
-		(property "Footprint" "Capacitor_SMD:C_0402_1005Metric_Pad0.74x0.62mm_HandSolder"
+		(property "Footprint" "Capacitor_SMD:C_0805_2012Metric_Pad1.18x1.45mm_HandSolder"
 			(at 141.9352 36.83 0)
 			(effects
@@
 			)
 		)
-		(property "Manufacturer Part Number" "CL05B104K05NNNC"
+		(property "Manufacturer Part Number" "CL21B104KACNFNC"
 			(at 140.97 33.02 0)
 			(effects
@@
 			)
 		)
-		(property "Footprint" "Capacitor_SMD:C_0402_1005Metric_Pad0.74x0.62mm_HandSolder"
+		(property "Footprint" "Capacitor_SMD:C_0805_2012Metric_Pad1.18x1.45mm_HandSolder"
 			(at 206.7052 39.37 0)
 			(effects
@@
 			)
 		)
-		(property "Manufacturer Part Number" "CL05B104KB5NFNC"
+		(property "Manufacturer Part Number" "CL21B104KBFXPJE"
 			(at 205.74 35.56 0)
 			(effects
@@
 			)
 		)
-		(property "Footprint" "Capacitor_SMD:C_0402_1005Metric_Pad0.74x0.62mm_HandSolder"
+		(property "Footprint" "Capacitor_SMD:C_0805_2012Metric_Pad1.18x1.45mm_HandSolder"
 			(at 228.2952 96.52 0)
 			(effects
@@
 			)
 		)
-		(property "Manufacturer Part Number" "CL05B223KB5NNNC"
+		(property "Manufacturer Part Number" "CL21B223JBANNNC"
 			(at 227.33 92.71 0)
 			(effects
@@
 			)
 		)
-		(property "Footprint" "Capacitor_SMD:C_0402_1005Metric_Pad0.74x0.62mm_HandSolder"
+		(property "Footprint" "Capacitor_SMD:C_0805_2012Metric_Pad1.18x1.45mm_HandSolder"
 			(at 232.1052 142.24 0)
 			(effects
@@
 			)
 		)
-		(property "Manufacturer Part Number" "CL05B223KB5NNNC"
+		(property "Manufacturer Part Number" "CL21B223JBANNNC"
 			(at 231.14 138.43 0)
 			(effects
@@
 			)
 		)
-		(property "Footprint" "Resistor_SMD:R_0402_1005Metric_Pad0.72x0.64mm_HandSolder"
+		(property "Footprint" "Resistor_SMD:R_0805_2012Metric_Pad1.20x1.40mm_HandSolder"
 			(at 210.312 142.24 90)
 			(effects
@@
 			)
 		)
-		(property "Footprint" "Capacitor_SMD:C_0402_1005Metric_Pad0.74x0.62mm_HandSolder"
+		(property "Footprint" "Capacitor_SMD:C_0805_2012Metric_Pad1.18x1.45mm_HandSolder"
 			(at 172.4152 66.04 0)
 			(effects
@@
 			)
 		)
-		(property "Manufacturer Part Number" "CL05B104K05NNNC"
+		(property "Manufacturer Part Number" "CL21B104KACNFNC"
 			(at 171.45 62.23 0)
 			(effects
