File: hardware/LCC_Booster/can_interface.kicad_sch (KiCad schematic)
At the start: 10 parts, among them U10 MCP2562-E-SN, U9 MCP2518FD-xQBB, Y1 ECS-400-20-46X

Commit message: Version 5 of PCB
Parts:
- C29, C30, C31: footprint Capacitor_SMD:C_0402_1005Metric_Pad0.74x0.62mm_HandSolder -> Capacitor_SMD:C_0805_2012Metric_Pad1.18x1.45mm_HandSolder
- C32, C33: footprint Capacitor_SMD:C_0402_1005Metric_Pad0.74x0.62mm_HandSolder -> Capacitor_SMD:C_0805_2012Metric_Pad1.18x1.45mm_HandSolder; Manufacturer Part Number CL05B104K05NNNC -> CL21B104KACNFNC
Changed lines of the file:
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@@
 	(title_block
 		(title "Arduino Nano LCC Booster")
-		(date "2024-09-10")
-		(rev "4")
+		(date "2024-11-16")
+		(rev "5")
 		(company "TMRC")
 		(comment 1 "Noah Paladino")
@@
 			)
 		)
-		(property "Footprint" "Capacitor_SMD:C_0402_1005Metric_Pad0.74x0.62mm_HandSolder"
+		(property "Footprint" "Capacitor_SMD:C_0805_2012Metric_Pad1.18x1.45mm_HandSolder"
 			(at 109.22 90.4748 0)
 			(effects
@@
 			)
 		)
-		(property "Footprint" "Capacitor_SMD:C_0402_1005Metric_Pad0.74x0.62mm_HandSolder"
+		(property "Footprint" "Capacitor_SMD:C_0805_2012Metric_Pad1.18x1.45mm_HandSolder"
 			(at 153.3652 60.96 0)
 			(effects
@@
 			)
 		)
-		(property "Footprint" "Capacitor_SMD:C_0402_1005Metric_Pad0.74x0.62mm_HandSolder"
+		(property "Footprint" "Capacitor_SMD:C_0805_2012Metric_Pad1.18x1.45mm_HandSolder"
 			(at 109.22 100.6348 0)
 			(effects
@@
 			)
 		)
-		(property "Footprint" "Capacitor_SMD:C_0402_1005Metric_Pad0.74x0.62mm_HandSolder"
+		(property "Footprint" "Capacitor_SMD:C_0805_2012Metric_Pad1.18x1.45mm_HandSolder"
 			(at 194.0052 60.96 0)
 			(effects
@@
 			)
 		)
-		(property "Manufacturer Part Number" "CL05B104K05NNNC"
+		(property "Manufacturer Part Number" "CL21B104KACNFNC"
 			(at 193.04 57.15 0)
 			(effects
@@
 			)
 		)
-		(property "Footprint" "Capacitor_SMD:C_0402_1005Metric_Pad0.74x0.62mm_HandSolder"
+		(property "Footprint" "Capacitor_SMD:C_0805_2012Metric_Pad1.18x1.45mm_HandSolder"
 			(at 166.0652 60.96 0)
 			(effects
@@
 			)
 		)
-		(property "Manufacturer Part Number" "CL05B104K05NNNC"
+		(property "Manufacturer Part Number" "CL21B104KACNFNC"
 			(at 165.1 57.15 0)
 			(effects
