File: hardware/LCC_Booster/dcc_isolator.kicad_sch (KiCad schematic)
At the start: 7 parts, among them U1 6N137, U2 6N137

Commit message: Add Fault Pin Inputs to Arduino
Other:
- company: (none) -> TMRC
- title: (none) -> Arduino Nano LCC Booster
Changed lines of the file:
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@@
 	(generator_version "8.0")
 	(paper "A4")
+	(title_block
+		(title "Arduino Nano LCC Booster")
+		(date "2024-09-10")
+		(rev "4")
+		(company "TMRC")
+		(comment 1 "Noah Paladino")
+	)
 	(junction
 		(at 124.46 85.09)

Commit message: Update for PCB Assembly
Parts:
- added R15: R2k 1W, Resistor_SMD:R_2512_6332Metric_Pad1.40x3.35mm_HandSolder, symbol Device:R
- C34, C35: MANUFACTURER (none) -> Samsung; Manufacturer Part Number (none) -> CL05B104K05NNNC
- R13: renamed from R14; footprint Resistor_SMD:R_01005_0402Metric_Pad0.57x0.30mm_HandSolder -> Resistor_SMD:R_0402_1005Metric_Pad0.72x0.64mm_HandSolder; MANUFACTURER (none) -> Yageo; Manufacturer Part Number (none) -> RC0402JR-7W10KL
- R14: renamed from R13; value R1k 2W -> R2k 1W; footprint Resistor_SMD:R_01005_0402Metric_Pad0.57x0.30mm_HandSolder -> Resistor_SMD:R_2512_6332Metric_Pad1.40x3.35mm_HandSolder; MANUFACTURER (none) -> Yageo; Manufacturer Part Number (none) -> AC2512JK-072KL
- R16: renamed from R15; footprint Resistor_SMD:R_01005_0402Metric_Pad0.57x0.30mm_HandSolder -> Resistor_SMD:R_0402_1005Metric_Pad0.72x0.64mm_HandSolder; MANUFACTURER (none) -> Yageo; Manufacturer Part Number (none) -> RC0402JR-7W10KL
- U11: renamed from U2; MANUFACTURER (none) -> Lite-On; Manufacturer Part Number (none) -> 6N137S-TA1-L
- U12: renamed from U1; MANUFACTURER (none) -> Lite-On; Manufacturer Part Number (none) -> 6N137S-TA1-L
Connections:
- net raw_dcc_p: now also R15.1
- net at R14.2, U11.3 (C), U12.2 (A): now also R15.2
Other:
- moved on the sheet: R14

Commit message: Version 5 of PCB
Parts:
- C34, C35: footprint Capacitor_SMD:C_0402_1005Metric_Pad0.74x0.62mm_HandSolder -> Capacitor_SMD:C_0805_2012Metric_Pad1.18x1.45mm_HandSolder; Manufacturer Part Number CL05B104K05NNNC -> CL21B104KACNFNC
- R13, R16: footprint Resistor_SMD:R_0402_1005Metric_Pad0.72x0.64mm_HandSolder -> Resistor_SMD:R_0805_2012Metric_Pad1.20x1.40mm_HandSolder; Manufacturer Part Number RC0402JR-7W10KL -> RC0805JR-0710KL
Changed lines of the file:
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@@
 	(title_block
 		(title "Arduino Nano LCC Booster")
-		(date "2024-09-10")
-		(rev "4")
+		(date "2024-11-16")
+		(rev "5")
 		(company "TMRC")
 		(comment 1 "Noah Paladino")
@@
 			)
 		)
-		(property "Footprint" "Capacitor_SMD:C_0402_1005Metric_Pad0.74x0.62mm_HandSolder"
+		(property "Footprint" "Capacitor_SMD:C_0805_2012Metric_Pad1.18x1.45mm_HandSolder"
 			(at 180.0352 64.77 0)
 			(effects
@@
 			)
 		)
-		(property "Manufacturer Part Number" "CL05B104K05NNNC"
+		(property "Manufacturer Part Number" "CL21B104KACNFNC"
 			(at 179.07 60.96 0)
 			(effects
@@
 			)
 		)
-		(property "Footprint" "Capacitor_SMD:C_0402_1005Metric_Pad0.74x0.62mm_HandSolder"
+		(property "Footprint" "Capacitor_SMD:C_0805_2012Metric_Pad1.18x1.45mm_HandSolder"
 			(at 116.5352 64.77 0)
 			(effects
@@
 			)
 		)
-		(property "Manufacturer Part Number" "CL05B104K05NNNC"
+		(property "Manufacturer Part Number" "CL21B104KACNFNC"
 			(at 115.57 60.96 0)
 			(effects
@@
 			)
 		)
-		(property "Footprint" "Resistor_SMD:R_0402_1005Metric_Pad0.72x0.64mm_HandSolder"
+		(property "Footprint" "Resistor_SMD:R_0805_2012Metric_Pad1.20x1.40mm_HandSolder"
 			(at 193.548 60.96 90)
 			(effects
@@
 			)
 		)
-		(property "Manufacturer Part Number" "RC0402JR-7W10KL"
+		(property "Manufacturer Part Number" "RC0805JR-0710KL"
 			(at 191.77 60.96 0)
 			(effects
@@
 			)
 		)
-		(property "Footprint" "Resistor_SMD:R_0402_1005Metric_Pad0.72x0.64mm_HandSolder"
+		(property "Footprint" "Resistor_SMD:R_0805_2012Metric_Pad1.20x1.40mm_HandSolder"
 			(at 107.188 60.96 90)
 			(effects
@@
 			)
 		)
-		(property "Manufacturer Part Number" "RC0402JR-7W10KL"
+		(property "Manufacturer Part Number" "RC0805JR-0710KL"
 			(at 105.41 60.96 0)
 			(effects
