File: hardware/LCC_Booster/LCC_Booster.kicad_pcb (KiCad board)
At the start: 2 copper layers, 90 x 100 mm, 84 parts, among them J1 A00-216-262-450, J2 54-00166, J3 Screw_Terminal_01x08, SW1 SW_Push, U1 6N137, U10 DRV8874PWPR, U11 MCP2518FD-xQBB, U12 MCP2562-E-SN, U2 6N137, U3 SN74HC253DR, U4 DRV8874PWPR, U5 SN74HC253DR, U6 DRV8874PWPR, U7 SN74HC253DR, U8 DRV8874PWPR, U9 SN74HC253DR, Y1 ECS-400-20-46X

Commit message: Update for PCB Assembly
Parts:
- removed the J1 at (100.0, 88.5)
- removed the JP1 at (91.0, 110.0)
- added J3: RJHSE508002, RJHSE508002:AMPHENOL_RJHSE508002, F.Cu at (105.0, 88.2)
- added R15: R2k 1W, Resistor_SMD:R_2512_6332Metric_Pad1.40x3.35mm_HandSolder, F.Cu at (67.0, 104.0)
- C11, C18, C25, C4: value C10u -> C10u VM
- C12, C19, C26, C5: value C100n -> C100n VM
- R1, R10, R4, R7: footprint Resistor_SMD:R_01005_0402Metric_Pad0.57x0.30mm_HandSolder -> Resistor_SMD:R_0805_2012Metric_Pad1.20x1.40mm_HandSolder
- R11, R12, R2, R3, R5, R6, R8, R9: footprint Resistor_SMD:R_01005_0402Metric_Pad0.57x0.30mm_HandSolder -> Resistor_SMD:R_0402_1005Metric_Pad0.72x0.64mm_HandSolder
- R13: renamed from R14; footprint Resistor_SMD:R_01005_0402Metric_Pad0.57x0.30mm_HandSolder -> Resistor_SMD:R_0402_1005Metric_Pad0.72x0.64mm_HandSolder
- R14: renamed from R13; value R1k 2W -> R2k 1W; footprint Resistor_SMD:R_01005_0402Metric_Pad0.57x0.30mm_HandSolder -> Resistor_SMD:R_2512_6332Metric_Pad1.40x3.35mm_HandSolder
- R16: renamed from R15; footprint Resistor_SMD:R_01005_0402Metric_Pad0.57x0.30mm_HandSolder -> Resistor_SMD:R_0402_1005Metric_Pad0.72x0.64mm_HandSolder
- moved R10 52.3 mm to (41.5, 35.2), turned to 0 degrees
- moved R7 40.8 mm to (41.5, 31.8), turned to 0 degrees
- moved R4 29.3 mm to (41.5, 28.2), turned to 0 degrees
- moved R1 17.9 mm to (41.5, 24.8), turned to 0 degrees
- moved R14 6.60 mm to (61.5, 104.0)
- moved U12 3.25 mm to (75.8, 99.2)
- moved R16 3.00 mm to (82.5, 99.2)
- moved C35 2.50 mm to (80.2, 93.2)
- moved C16 0.33 mm to (46.0, 72.2)
- moved C23 0.33 mm to (46.0, 87.2)
- moved C9 0.33 mm to (46.0, 57.2)
- moved C2 0.17 mm to (45.5, 42.2)
- moved R12 0.15 mm to (55.0, 88.4)
- moved R3 0.15 mm to (55.0, 43.4)
- moved R6 0.15 mm to (55.0, 58.4)
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- renumbered J3 to J1, JP2 to JP1, JP8 to JP10, JP9 to JP11, JP3 to JP2, JP10 to JP3, JP11 to JP4, JP12 to JP5, JP4 to JP6, JP5 to JP7, JP6 to JP8, JP7 to JP9, U3 to U1, U12 to U10, U2 to U11, U1 to U12, U4 to U2, U5 to U3, U6 to U4, U7 to U5, U8 to U6, U9 to U7, U10 to U8, U11 to U9
Routing:
- net /can_shield: track 74.4 -> 16.6 mm
- net /raw_dcc_p: track 111.5 -> 154.1 mm, vias 1 -> 2
- net GND: track 324.3 -> 290.1 mm, vias 74 -> 79
- net /out2_D: track 21.3 -> 51.1 mm
- net IOREF: track 271.3 -> 289.0 mm, vias 18 -> 19
- net /out2_C: track 19.3 -> 34.7 mm
- net /nFault_A: track 13.8 -> 28.3 mm, vias 1 -> 2
- net /raw_dcc_n: track 129.9 -> 142.9 mm
- net Net-(U11-C): track 22.0 -> 33.9 mm
- net /out2_B: track 19.1 -> 30.0 mm
- net /can_l: track 30.8 -> 41.2 mm
- net /out2_A: track 21.2 -> 29.1 mm
- net /can_h: track 33.2 -> 40.9 mm
- net /nFault_B: track 37.3 -> 43.5 mm, vias 1 -> 2
- net /nFault_C: track 77.6 -> 82.5 mm, vias 2 -> 3
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
Commit message: Version 5 of PCB
Parts:
- C1, C10, C12, C13, C14, C15, C16, C17, C19, C2, C20, C21, C22, C23, C24, C26, C27, C28, C29, C3, C30, C31, C32, C33, C34, C35, C5, C6, C7, C8, C9: footprint Capacitor_SMD:C_0402_1005Metric_Pad0.74x0.62mm_HandSolder -> Capacitor_SMD:C_0805_2012Metric_Pad1.18x1.45mm_HandSolder
- R11, R12, R13, R16, R2, R3, R5, R6, R8, R9: footprint Resistor_SMD:R_0402_1005Metric_Pad0.72x0.64mm_HandSolder -> Resistor_SMD:R_0805_2012Metric_Pad1.20x1.40mm_HandSolder
- moved R11 3.98 mm to (49.5, 85.8)
- moved R2 3.98 mm to (49.5, 40.8)
- moved R5 3.98 mm to (49.5, 55.8)
- moved R8 3.98 mm to (49.5, 70.8)
- moved R12 2.11 mm to (53.5, 87.0)
- moved R3 2.11 mm to (53.5, 42.0)
- moved R6 2.11 mm to (53.5, 57.0)
- moved R9 2.11 mm to (53.5, 72.0)
- moved C29 1.99 mm to (99.0, 70.0)
- moved C12 1.80 mm to (40.2, 68.3)
- moved C19 1.80 mm to (40.2, 83.3)
- moved C26 1.80 mm to (40.2, 98.3)
- moved C5 1.80 mm to (40.2, 53.3)
- moved C13 1.68 mm to (45.8, 66.7)
- moved C20 1.68 mm to (45.8, 81.7)
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Routing:
- net GND: track 290.1 -> 229.5 mm, vias 79 -> 136
- net VTRACK: track 105.0 -> 146.2 mm, vias 4 -> 12
- net /out2_D: track 51.1 -> 19.0 mm
- net /out2_C: track 34.7 -> 15.9 mm
- net /raw_dcc_p: track 154.1 -> 136.9 mm
- net IOREF: track 289.0 -> 303.8 mm, vias 19 -> 20
- net /out2_B: track 30.0 -> 16.8 mm
- net /pwm_B: track 65.5 -> 52.7 mm
- net /out2_A: track 29.1 -> 18.8 mm
- net /pwm_A: track 69.6 -> 60.3 mm, vias 1 -> 3
- net /sense_C: track 80.0 -> 75.3 mm
- net /pwm_D: track 70.7 -> 66.1 mm
- net /pwm_C: track 65.6 -> 62.4 mm
- net +5V: track 89.0 -> 92.0 mm
- net /sense_A: track 62.4 -> 59.5 mm
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Other:
- board text added: "TMRC System 4 Block Card v5"
- board text removed: "TMRC System 4 Block Card v4"

Commit message: Added location holes to solder paste template
Parts:
- H1, H2, H3, H4: footprint MountingHole:MountingHole_4.3mm_M4_Pad_Via -> MountingHoles:MountingHole_4.3mm_M4_Pad_Via_PasteAlign

Commit message: PicoLCC
Routing:
- net /can_h: track 40.3 -> 37.6 mm
Changed lines of the file:
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@@
-	)
-	(segment
-		(start 102.46 93.137)
-		(end 102.612 93.289)
-		(width 0.2)
-		(layer "B.Cu")
-		(net 38)
 	)
 	(segment
@@
 	)
 	(segment
-		(start 101.924264 75.75)
-		(end 100.98 76.694264)
+		(start 103 75.75)
+		(end 102.46 76.29)
 		(width 0.2)
 		(layer "B.Cu")
@@
 	)
 	(segment
-		(start 103 75.75)
-		(end 101.924264 75.75)
+		(start 102.46 93.137)
+		(end 102.612 93.289)
 		(width 0.2)
 		(layer "B.Cu")
@@
 	)
 	(segment
-		(start 100.98 76.803)
-		(end 101 76.823)
-		(width 0.2)
-		(layer "B.Cu")
-		(net 38)
-	)
-	(segment
-		(start 100.98 76.694264)
-		(end 100.98 76.803)
-		(width 0.2)
-		(layer "B.Cu")
-		(net 38)
-	)
-	(segment
-		(start 101 76.823)
+		(start 102.46 76.29)
 		(end 102.46 76.823)
 		(width 0.2)
