File: hardware/Pico_LCC/Pico_LCC.kicad_sch (KiCad schematic)
At the start: 7 parts, among them J1 Screw_Terminal_01x08, J2 RJHSE508002, U1 Pico

Commit message: PicoLCC
Parts:
- added J3: SM04B-SRSS-TB, SM04B_SRSS_TB:CONN_SM04B-SRSS-TB_JST, symbol SM04B_SRSS_TB:SM04B-SRSS-TB
- added JP1: SolderJumper_2_Open, Jumper:SolderJumper-2_P1.3mm_Open_RoundedPad1.0x1.5mm, symbol Jumper:SolderJumper_2_Open
- added R12, R9: R2.2k, Resistor_SMD:R_0805_2012Metric_Pad1.20x1.40mm_HandSolder, symbol Device:R
- added U14: SN3257QPWRQ1, SN3257QPWRQ1:SOIC_PRQ1_TEX, symbol SN3257QPWRQ1:SN3257QPWRQ1
- J1: value Screw_Terminal_01x08 -> Screw_Terminal_01x12
Connections:
- net +3.3V: now also J3.2, R12.1, R9.1, U14.16 (VDD)
- net GND: now also J3.1, JP1.2 (B), U14.10 (S3B), U14.11 (S3A), U14.15 (~{EN}), U14.5 (S2A), U14.6 (S2B), U14.8 (GND)
- net can_shield: now also JP1.1 (A)
- net cs-canrx: now also U1.22 (GPIO17)
- net dcc_en_A: now also U1.2 (GPIO1)
- net dcc_en_B: now also U1.7 (GPIO5)
- net dcc_en_C: now also U1.12 (GPIO9)
- net dcc_en_D: now also U1.17 (GPIO13)
- net dir_A: now also U1.4 (GPIO2)
- net dir_B: now also U1.9 (GPIO6)
- net dir_C: now also U1.14 (GPIO10)
- net dir_D: now also U1.19 (GPIO14)
- net int-cantx: now also U1.29 (GPIO22)
- net nFault_A: now also U1.1 (GPIO0)
- net nFault_B: now also U1.6 (GPIO4)
- net nFault_C: now also U1.11 (GPIO8)
- net nFault_D: now also U1.16 (GPIO12)
- net pwm_A: now also U1.5 (GPIO3)
- net pwm_B: now also U1.10 (GPIO7)
- net pwm_C: now also U1.15 (GPIO11)
- net pwm_D: now also U1.20 (GPIO15)
- net sense_A: now also U14.2 (S1A)
- net sense_B: now also U14.3 (S1B)
- net sense_C: now also U14.14 (S4A)
- net sense_D: now also U14.13 (S4B)
- net cipo: now reaches U1.21 (GPIO16)
- net sck: now reaches U1.24 (GPIO18)
- net copi: now reaches U1.25 (GPIO19)
- net sda: now reaches U1.26 (GPIO20)
- net sda: now also J3.3, R12.2
- net scl: now reaches U1.27 (GPIO21)
- net scl: now also J3.4, R9.2
- net adc0: now reaches U1.31 (GPIO26_ADC0)
- net adc0: now also U14.4 (D1)
- net adc1: now reaches U1.32 (GPIO27_ADC1)
- net adc1: now also U14.12 (D4)
- net adc_sel: now reaches U1.34 (GPIO28_ADC2)
- net adc_sel: now also U14.1 (SEL)
- net can_h renamed can_h+
- net can_l renamed can_l-
- no-connect marks 7 -> 13
Other:
- sheet CAN Interface ports: added can_h+, can_l-; removed can_h, can_l
- company: (none) -> TMRC
- title: (none) -> Raspberry Pi Pico LCC Block Card
- moved on the sheet: H1, H2, H3, H4, J1, J2A, J2B, U1
