File: hardware/Pico_LCC/block_driver.kicad_sch (KiCad schematic)
At the start: 11 parts, among them U2 SN74HC253DR, U3 DRV8874PWPR

Commit message: PicoLCC
Parts:
- renumbered C3 to C10, C4 to C11, C5 to C12, C6 to C13, C7 to C14, C1 to C8, C2 to C9, R1 to R4, R2 to R5, U2 to U4, U3 to U5
Other:
- title: Arduino Nano LCC Booster -> Raspberry Pi Pico LCC Block Card
Changed lines of the file:
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@@
 	(generator "eeschema")
 	(generator_version "8.0")
-	(paper "A4")
+	(paper "USLetter")
 	(title_block
-		(title "Arduino Nano LCC Booster")
-		(date "2024-11-16")
-		(rev "5")
+		(title "Raspberry Pi Pico LCC Block Card")
+		(date "2025-01-09")
+		(rev "1")
 		(company "TMRC")
 		(comment 1 "Noah Paladino")
@@
 		(dnp no)
 		(fields_autoplaced yes)
-		(property "Reference" "R2"
+		(property "Reference" "R5"
 			(at 203.2 135.8899 0)
 			(effects
@@
 		(dnp no)
 		(fields_autoplaced yes)
-		(property "Reference" "C2"
+		(property "Reference" "C9"
 			(at 156.21 101.5999 0)
 			(effects
@@
 		(dnp no)
 		(fields_autoplaced yes)
-		(property "Reference" "R1"
+		(property "Reference" "R4"
 			(at 161.29 57.1499 0)
 			(effects
@@
 		(dnp no)
 		(fields_autoplaced yes)
-		(property "Reference" "#PWR08"
+		(property "Reference" "#PWR016"
 			(at 189.23 34.29 0)
 			(effects
@@
 		(dnp no)
 		(fields_autoplaced yes)
-		(property "Reference" "#PWR05"
+		(property "Reference" "#PWR013"
 			(at 123.19 30.48 0)
 			(effects
@@
 		(dnp no)
 		(fields_autoplaced yes)
-		(property "Reference" "U2"
+		(property "Reference" "U4"
 			(at 92.71 50.8 0)
 			(effects
@@
 		(on_board yes)
 		(dnp no)
-		(property "Reference" "#PWR06"
+		(property "Reference" "#PWR014"
 			(at 140.97 44.45 0)
 			(effects
@@
 		(dnp no)
 		(fields_autoplaced yes)
-		(property "Reference" "C4"
+		(property "Reference" "C11"
 			(at 193.04 34.2899 0)
 			(effects
@@
 		(on_board yes)
 		(dnp no)
-		(property "Reference" "#PWR04"
+		(property "Reference" "#PWR012"
 			(at 90.17 97.79 0)
 			(effects
@@
 		(on_board yes)
 		(dnp no)
-		(property "Reference" "#PWR09"
+		(property "Reference" "#PWR017"
 			(at 196.85 48.26 0)
 			(effects
@@
 		(dnp no)
 		(fields_autoplaced yes)
-		(property "Reference" "C1"
+		(property "Reference" "C8"
 			(at 144.78 31.7499 0)
 			(effects
@@
 		(dnp no)
 		(fields_autoplaced yes)
-		(property "Reference" "C5"
+		(property "Reference" "C12"
 			(at 209.55 34.2899 0)
 			(effects
@@
 		(dnp no)
 		(fields_autoplaced yes)
-		(property "Reference" "C6"
+		(property "Reference" "C13"
 			(at 231.14 91.4399 0)
 			(effects
@@
 		(dnp no)
 		(fields_autoplaced yes)
-		(property "Reference" "#PWR07"
+		(property "Reference" "#PWR015"
 			(at 156.21 115.57 0)
 			(effects
@@
 		(dnp no)
 		(fields_autoplaced yes)
-		(property "Reference" "#PWR010"
+		(property "Reference" "#PWR018"
 			(at 200.66 160.02 0)
 			(effects
@@
 		(dnp no)
 		(fields_autoplaced yes)
-		(property "Reference" "#PWR011"
+		(property "Reference" "#PWR019"
 			(at 240.03 121.92 0)
 			(effects
@@
 		(dnp no)
 		(fields_autoplaced yes)
-		(property "Reference" "C7"
+		(property "Reference" "C14"
 			(at 234.95 135.8899 0)
 			(effects
@@
 		(dnp no)
 		(fields_autoplaced yes)
-		(property "Reference" "C3"
+		(property "Reference" "C10"
 			(at 175.26 60.9599 0)
 			(effects
@@
 		(dnp no)
 		(fields_autoplaced yes)
-		(property "Reference" "U3"
+		(property "Reference" "U5"
 			(at 200.66 48.26 0)
 			(effects
