File: hardware/Pico_LCC/can_interface.kicad_sch (KiCad schematic)
At the start: 10 parts, among them U10 MCP2518FD-xQBB, U11 MCP2562-E-SN, Y1 ECS-400-20-46X

Commit message: PicoLCC
Connections:
- net at JP6.1 (A): now also U10.1 (TXCAN), U11.1 (TXD); no longer U10.4 (~{INT})
- net at JP5.1 (A): now also U10.2 (RXCAN), U11.4 (RXD); no longer U10.13 (~{CS})
- net can_h renamed can_h+
- net can_l renamed can_l-
- new net: JP6.3 (B), U10.4 (~{INT})
- new net: JP5.3 (B), U10.13 (~{CS})
Other:
- title: Arduino Nano LCC Booster -> Raspberry Pi Pico LCC Block Card
- moved on the sheet: C29, C30, Y1
Changed lines of the file:
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@@
 	(generator "eeschema")
 	(generator_version "8.0")
-	(paper "A4")
+	(paper "USLetter")
 	(title_block
-		(title "Arduino Nano LCC Booster")
-		(date "2024-11-16")
-		(rev "5")
+		(title "Raspberry Pi Pico LCC Block Card")
+		(date "2025-01-09")
+		(rev "1")
 		(company "TMRC")
 		(comment 1 "Noah Paladino")
+	)
+	(junction
+		(at 109.22 90.17)
+		(diameter 0)
+		(color 0 0 0 0)
 	)
 	(junction
@@
 	)
 	(junction
-		(at 109.22 91.44)
+		(at 96.52 100.33)
+		(diameter 0)
+		(color 0 0 0 0)
+	)
+	(junction
+		(at 109.22 100.33)
 		(diameter 0)
 		(color 0 0 0 0)
@@
 	)
 	(junction
-		(at 96.52 101.6)
-		(diameter 0)
-		(color 0 0 0 0)
-	)
-	(junction
 		(at 146.05 53.34)
 		(diameter 0)
@@
 	)
 	(junction
-		(at 109.22 101.6)
-		(diameter 0)
-		(color 0 0 0 0)
-	)
-	(junction
 		(at 186.69 123.19)
 		(diameter 0)
@@
 	(wire
 		(pts
-			(xy 96.52 91.44) (xy 96.52 101.6)
-		)
-		(stroke
-			(width 0)
-			(type default)
-		)
-	)
-	(wire
-		(pts
-			(xy 115.57 92.71) (xy 115.57 101.6)
+			(xy 96.52 90.17) (xy 96.52 100.33)
+		)
+		(stroke
+			(width 0)
+			(type default)
+		)
+	)
+	(wire
+		(pts
+			(xy 115.57 92.71) (xy 115.57 100.33)
 		)
 		(stroke
@@
 	(wire
 		(pts
+			(xy 106.68 90.17) (xy 109.22 90.17)
+		)
+		(stroke
+			(width 0)
+			(type default)
+		)
+	)
+	(wire
+		(pts
 			(xy 186.69 48.26) (xy 186.69 53.34)
 		)
@@
 	(wire
 		(pts
-			(xy 96.52 101.6) (xy 96.52 123.19)
-		)
-		(stroke
-			(width 0)
-			(type default)
-		)
-	)
-	(wire
-		(pts
-			(xy 109.22 101.6) (xy 115.57 101.6)
+			(xy 109.22 100.33) (xy 115.57 100.33)
 		)
 		(stroke
@@
 	(wire
 		(pts
-			(xy 160.02 85.09) (xy 158.75 85.09)
+			(xy 161.29 85.09) (xy 158.75 85.09)
 		)
 		(stroke
@@
 	(wire
 		(pts
+			(xy 96.52 100.33) (xy 96.52 123.19)
+		)
+		(stroke
+			(width 0)
+			(type default)
+		)
+	)
+	(wire
+		(pts
 			(xy 104.14 73.66) (xy 104.14 82.55)
 		)
@@
 	(wire
 		(pts
-			(xy 101.6 91.44) (xy 96.52 91.44)
-		)
-		(stroke
-			(width 0)
-			(type default)
-		)
-	)
-	(wire
-		(pts
-			(xy 109.22 91.44) (xy 109.22 90.17)
+			(xy 99.06 90.17) (xy 96.52 90.17)
 		)
 		(stroke
@@
 	(wire
 		(pts
+			(xy 106.68 100.33) (xy 109.22 100.33)
+		)
+		(stroke
+			(width 0)
+			(type default)
+		)
+	)
+	(wire
+		(pts
 			(xy 96.52 123.19) (xy 133.35 123.19)
 		)
@@
 	(wire
 		(pts
-			(xy 96.52 101.6) (xy 101.6 101.6)
+			(xy 96.52 100.33) (xy 99.06 100.33)
 		)
 		(stroke
@@
 		)
 	)
-	(hierarchical_label "can_h"
+	(hierarchical_label "can_h+"
 		(shape bidirectional)
 		(at 207.01 77.47 0)
@@
 		)
 	)
-	(hierarchical_label "can_l"
+	(hierarchical_label "can_l-"
 		(shape bidirectional)
 		(at 207.01 82.55 0)
@@
 	(hierarchical_label "int-cantx"
 		(shape bidirectional)
-		(at 160.02 85.09 270)
+		(at 161.29 85.09 270)
 		(fields_autoplaced yes)
 		(effects
@@
 	(symbol
 		(lib_id "Device:C")
-		(at 105.41 91.44 90)
+		(at 102.87 90.17 90)
 		(unit 1)
 		(exclude_from_sim no)
@@
 		(dnp yes)
 		(property "Reference" "C29"
-			(at 105.41 94.742 90)
+			(at 102.87 93.472 90)
 			(effects
 				(font
@@
 		)
 		(property "Value" "C22p"
-			(at 105.41 97.282 90)
+			(at 102.87 96.012 90)
 			(effects
 				(font
@@
 		)
 		(property "Footprint" "Capacitor_SMD:C_0805_2012Metric_Pad1.18x1.45mm_HandSolder"
-			(at 109.22 90.4748 0)
+			(at 106.68 89.2048 0)
 			(effects
 				(font
@@
 		)
 		(property "Datasheet" "~"
-			(at 105.41 91.44 0)
+			(at 102.87 90.17 0)
 			(effects
 				(font
@@
 		)
 		(property "Description" "Unpolarized capacitor"
-			(at 105.41 91.44 0)
+			(at 102.87 90.17 0)
 			(effects
 				(font
@@
 		)
 		(property "Manufacturer Part Number" ""
-			(at 105.41 91.44 0)
+			(at 102.87 90.17 0)
 			(effects
 				(font
@@
 		(lib_id "Jumper:SolderJumper_3_Bridged12")
 		(at 154.94 85.09 90)
+		(mirror x)
 		(unit 1)
 		(exclude_from_sim yes)
@@
 		(dnp no)
 		(property "Reference" "JP6"
-			(at 152.4 86.3601 0)
+			(at 152.4 83.8199 0)
 			(effects
 				(font
@@
 		)
 		(property "Value" "SolderJumper_3_Bridged12"
-			(at 152.4 83.8201 90)
+			(at 152.4 86.3599 90)
 			(effects
 				(font
@@
 		(lib_id "Jumper:SolderJumper_3_Bridged12")
 		(at 104.14 68.58 270)
-		(mirror x)
 		(unit 1)
 		(exclude_from_sim yes)
@@
 		(dnp no)
 		(property "Reference" "JP5"
-			(at 106.68 69.8501 0)
+			(at 106.68 67.3099 0)
 			(effects
 				(font
@@
 		)
 		(property "Value" "SolderJumper_3_Bridged12"
-			(at 106.68 67.3101 90)
+			(at 106.68 69.8499 90)
 			(effects
 				(font
@@
 	(symbol
 		(lib_id "ECS-400-20-46X:ECS-400-20-46X")
-		(at 109.22 96.52 90)
+		(at 109.22 95.25 90)
 		(unit 1)
 		(exclude_from_sim no)
@@
 		(on_board yes)
 		(dnp yes)
-		(fields_autoplaced yes)
 		(property "Reference" "Y1"
-			(at 111.76 95.2499 90)
+			(at 111.76 93.9799 90)
 			(effects
 				(font
@@
 		)
 		(property "Value" "ECS-400-20-46X"
-			(at 111.76 97.7899 90)
+			(at 113.03 95.504 0)
 			(effects
 				(font
@@
 		)
 		(property "Footprint" "ECS_400_20_46X:XTAL_ECS-400-20-46X"
-			(at 109.22 96.52 0)
+			(at 109.22 95.25 0)
 			(effects
 				(font
@@
 		)
 		(property "Datasheet" ""
-			(at 109.22 96.52 0)
+			(at 109.22 95.25 0)
 			(effects
 				(font
@@
 		)
 		(property "Description" ""
-			(at 109.22 96.52 0)
+			(at 109.22 95.25 0)
 			(effects
 				(font
@@
 		)
 		(property "MANUFACTURER" "ECS Inc."
-			(at 109.22 96.52 0)
+			(at 109.22 95.25 0)
 			(effects
 				(font
@@
 		)
 		(property "STANDARD" "IPC-7251"
-			(at 109.22 96.52 0)
+			(at 109.22 95.25 0)
 			(effects
 				(font
@@
 		)
 		(property "Manufacturer Part Number" ""
-			(at 109.22 96.52 0)
+			(at 109.22 95.25 0)
 			(effects
 				(font
@@
 	(symbol
 		(lib_id "Device:C")
-		(at 105.41 101.6 90)
+		(at 102.87 100.33 90)
 		(unit 1)
 		(exclude_from_sim no)
@@
 		(dnp yes)
 		(property "Reference" "C30"
-			(at 105.41 104.902 90)
+			(at 102.87 103.632 90)
 			(effects
 				(font
@@
 		)
 		(property "Value" "C22p"
-			(at 105.41 107.442 90)
+			(at 102.87 106.172 90)
 			(effects
 				(font
@@
 		)
 		(property "Footprint" "Capacitor_SMD:C_0805_2012Metric_Pad1.18x1.45mm_HandSolder"
-			(at 109.22 100.6348 0)
+			(at 106.68 99.3648 0)
 			(effects
 				(font
@@
 		)
 		(property "Datasheet" "~"
-			(at 105.41 101.6 0)
+			(at 102.87 100.33 0)
 			(effects
 				(font
@@
 		)
 		(property "Description" "Unpolarized capacitor"
-			(at 105.41 101.6 0)
+			(at 102.87 100.33 0)
 			(effects
 				(font
@@
 		)
 		(property "Manufacturer Part Number" ""
-			(at 105.41 101.6 0)
-			(effects
-				(font
+			(at 102.87 100.33 0)
+			(effects
+				(font
