File: hardware/Pico_LCC/dcc_isolator.kicad_sch (KiCad schematic)
At the start: 8 parts, among them U12 6N137, U13 6N137

Commit message: PicoLCC
Other:
- title: Arduino Nano LCC Booster -> Raspberry Pi Pico LCC Block Card
Changed lines of the file:
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@@
 	(generator "eeschema")
 	(generator_version "8.0")
-	(paper "A4")
+	(paper "USLetter")
 	(title_block
-		(title "Arduino Nano LCC Booster")
-		(date "2024-11-16")
-		(rev "5")
+		(title "Raspberry Pi Pico LCC Block Card")
+		(date "2025-01-09")
+		(rev "1")
 		(company "TMRC")
 		(comment 1 "Noah Paladino")
